File: eagle/dmx reciever platine universal.sch (EAGLE design)
At the start: 23 parts, among them IC1 MEGA8515-P, IC3 7805T, IC4 75176AP, Q1 6MHz

Commit message: new output connector
Parts:
- removed U$2: 1X3, stiftleisten:1X3
- added X1: (no value), con-wago:233-112
Connections:
- net N$31 renamed OUTPUT4
- net N$32 renamed OUTPUT5
- net N$33 renamed OUTPUT6
- net N$34 renamed OUTPUT7
- net N$35 renamed OUTPUT8
- removed net N$13: IC4.B, U$2.1
- removed net N$24: IC4.A, U$2.2
- removed net N$28: IC1.(AD7)PA7, OUTPUTS.1
- removed net N$29: IC1.(AD6)PA6, OUTPUTS.2
- removed net N$30: IC1.(AD5)PA5, OUTPUTS.3
- removed net N$36: IC4.GND, U$2.3
- new net DMX+: IC4.A, X1.-8, X1.B-8
- new net DMX-: IC4.B, X1.-9, X1.B-9
- new net MOTOR+: X1.-11, X1.B-11
- new net MOTOR-: X1.-12, X1.B-12
- new net OUTPUT1: IC1.(AD7)PA7, OUTPUTS.1, X1.-6, X1.B-6
- new net OUTPUT2: IC1.(AD6)PA6, OUTPUTS.2, X1.-4, X1.B-4
- new net OUTPUT3: IC1.(AD5)PA5, OUTPUTS.3, X1.-2, X1.B-2
- net GND: now also IC4.GND, X1.-1, X1.-10, X1.-3, X1.-5, X1.-7, X1.B-1, X1.B-10, X1.B-3, X1.B-5, X1.B-7
Changed lines of the file:
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@@
 <?xml version="1.0" encoding="utf-8"?>
 <!DOCTYPE eagle SYSTEM "eagle.dtd">
-<eagle version="6.6.0">
+<eagle version="6.4">
 <drawing>
 <settings>
@@
 <part name="C6" library="rcl" deviceset="CPOL-EU" device="E3.5-8"/>
 <part name="IC4" library="751xx" deviceset="75176A" device="P"/>
-<part name="U$2" library="stiftleisten" deviceset="1X3" device=""/>
+<part name="X1" library="con-wago" deviceset="233-112" device=""/>
+<part name="GND2" library="supply1" deviceset="GND" device=""/>
 </parts>
 <sheets>
@@
 <instance part="C6" gate="G$1" x="93.98" y="-43.18"/>
 <instance part="IC4" gate="G$1" x="99.06" y="-20.32"/>
-<instance part="U$2" gate="G$1" x="134.62" y="-20.32"/>
+<instance part="X1" gate="G$1" x="104.14" y="-93.98"/>
+<instance part="GND2" gate="1" x="55.88" y="-111.76"/>
 </instances>
 <busses>
@@
 <wire x1="-2.54" y1="35.56" x2="-2.54" y2="38.1" width="0.1524" layer="91"/>
 </segment>
+<segment>
+<pinref part="X1" gate="G$1" pin="B-1"/>
+<wire x1="96.52" y1="-81.28" x2="55.88" y2="-81.28" width="0.1524" layer="91"/>
+<wire x1="55.88" y1="-81.28" x2="55.88" y2="-86.36" width="0.1524" layer="91"/>
+<pinref part="GND2" gate="1" pin="GND"/>
+<pinref part="X1" gate="G$1" pin="B-3"/>
+<wire x1="55.88" y1="-86.36" x2="55.88" y2="-91.44" width="0.1524" layer="91"/>
+<wire x1="55.88" y1="-96.52" x2="55.88" y2="-104.14" width="0.1524" layer="91"/>
+<wire x1="55.88" y1="-104.14" x2="55.88" y2="-109.22" width="0.1524" layer="91"/>
+<wire x1="96.52" y1="-86.36" x2="55.88" y2="-86.36" width="0.1524" layer="91"/>
+<junction x="55.88" y="-86.36"/>
+<pinref part="X1" gate="G$1" pin="B-5"/>
+<wire x1="96.52" y1="-91.44" x2="55.88" y2="-91.44" width="0.1524" layer="91"/>
+<wire x1="55.88" y1="-91.44" x2="55.88" y2="-96.52" width="0.1524" layer="91"/>
+<pinref part="X1" gate="G$1" pin="B-7"/>
+<wire x1="96.52" y1="-96.52" x2="55.88" y2="-96.52" width="0.1524" layer="91"/>
+<junction x="55.88" y="-96.52"/>
+<pinref part="X1" gate="G$1" pin="B-10"/>
+<wire x1="96.52" y1="-104.14" x2="55.88" y2="-104.14" width="0.1524" layer="91"/>
+<junction x="55.88" y="-104.14"/>
+<pinref part="X1" gate="G$1" pin="-1"/>
+<wire x1="96.52" y1="-81.28" x2="99.06" y2="-81.28" width="0.1524" layer="91"/>
+<junction x="96.52" y="-81.28"/>
+<pinref part="X1" gate="G$1" pin="-3"/>
+<wire x1="96.52" y1="-86.36" x2="99.06" y2="-86.36" width="0.1524" layer="91"/>
+<junction x="96.52" y="-86.36"/>
+<pinref part="X1" gate="G$1" pin="-5"/>
+<wire x1="99.06" y1="-91.44" x2="96.52" y2="-91.44" width="0.1524" layer="91"/>
+<junction x="96.52" y="-91.44"/>
+<pinref part="X1" gate="G$1" pin="-7"/>
+<wire x1="99.06" y1="-96.52" x2="96.52" y2="-96.52" width="0.1524" layer="91"/>
+<junction x="96.52" y="-96.52"/>
+<pinref part="X1" gate="G$1" pin="-10"/>
+<wire x1="99.06" y1="-104.14" x2="96.52" y2="-104.14" width="0.1524" layer="91"/>
+<junction x="96.52" y="-104.14"/>
+</segment>
+<segment>
+<pinref part="IC4" gate="G$1" pin="GND"/>
+<wire x1="111.76" y1="-27.94" x2="129.54" y2="-27.94" width="0.1524" layer="91"/>
+<label x="129.54" y="-27.94" size="1.778" layer="95" xref="yes"/>
+</segment>
 </net>
 <net name="N$11" class="0">
@@
 </segment>
 </net>
-<net name="N$28" class="0">
+<net name="OUTPUT1" class="0">
+<segment>
+<pinref part="X1" gate="G$1" pin="B-6"/>
+<wire x1="96.52" y1="-93.98" x2="81.28" y2="-93.98" width="0.1524" layer="91"/>
+<label x="81.28" y="-93.98" size="1.778" layer="95" rot="R180" xref="yes"/>
+<pinref part="X1" gate="G$1" pin="-6"/>
+<wire x1="96.52" y1="-93.98" x2="99.06" y2="-93.98" width="0.1524" layer="91"/>
+<junction x="96.52" y="-93.98"/>
+</segment>
 <segment>
 <pinref part="IC1" gate="G$1" pin="(AD7)PA7"/>
@@
 </segment>
 </net>
-<net name="N$29" class="0">
+<net name="OUTPUT2" class="0">
 <segment>
 <pinref part="IC1" gate="G$1" pin="(AD6)PA6"/>
@@
 <wire x1="66.04" y1="88.9" x2="127" y2="88.9" width="0.1524" layer="91"/>
 </segment>
-</net>
-<net name="N$30" class="0">
+<segment>
+<pinref part="X1" gate="G$1" pin="B-4"/>
+<wire x1="96.52" y1="-88.9" x2="81.28" y2="-88.9" width="0.1524" layer="91"/>
+<label x="81.28" y="-88.9" size="1.778" layer="95" rot="R180" xref="yes"/>
+<pinref part="X1" gate="G$1" pin="-4"/>
+<wire x1="99.06" y1="-88.9" x2="96.52" y2="-88.9" width="0.1524" layer="91"/>
+<junction x="96.52" y="-88.9"/>
+</segment>
+</net>
+<net name="OUTPUT3" class="0">
 <segment>
 <pinref part="IC1" gate="G$1" pin="(AD5)PA5"/>
@@
 <wire x1="66.04" y1="86.36" x2="127" y2="86.36" width="0.1524" layer="91"/>
 </segment>
-</net>
-<net name="N$31" class="0">
+<segment>
+<pinref part="X1" gate="G$1" pin="B-2"/>
+<wire x1="96.52" y1="-83.82" x2="81.28" y2="-83.82" width="0.1524" layer="91"/>
+<label x="81.28" y="-83.82" size="1.778" layer="95" rot="R180" xref="yes"/>
+<pinref part="X1" gate="G$1" pin="-2"/>
+<wire x1="99.06" y1="-83.82" x2="96.52" y2="-83.82" width="0.1524" layer="91"/>
+<junction x="96.52" y="-83.82"/>
+</segment>
+</net>
+<net name="OUTPUT4" class="0">
 <segment>
 <pinref part="IC1" gate="G$1" pin="(AD4)PA4"/>
@@
 </segment>
 </net>
-<net name="N$32" class="0">
+<net name="OUTPUT5" class="0">
 <segment>
 <pinref part="IC1" gate="G$1" pin="(AD3)PA3"/>
@@
 </segment>
 </net>
-<net name="N$33" class="0">
+<net name="OUTPUT6" class="0">
 <segment>
 <pinref part="IC1" gate="G$1" pin="(AD2)PA2"/>
@@
 </segment>
 </net>
-<net name="N$34" class="0">
+<net name="OUTPUT7" class="0">
 <segment>
 <pinref part="IC1" gate="G$1" pin="(AD1)PA1"/>
@@
 </segment>
 </net>
-<net name="N$35" class="0">
+<net name="OUTPUT8" class="0">
 <segment>
 <pinref part="IC1" gate="G$1" pin="(AD0)PA0"/>
@@
 </segment>
 </net>
-<net name="N$36" class="0">
-<segment>
-<pinref part="IC4" gate="G$1" pin="GND"/>
-<pinref part="U$2" gate="G$1" pin="3"/>
-<wire x1="111.76" y1="-27.94" x2="129.54" y2="-27.94" width="0.1524" layer="91"/>
-</segment>
-</net>
-<net name="N$13" class="0">
+<net name="DMX+" class="0">
+<segment>
+<pinref part="X1" gate="G$1" pin="B-8"/>
+<wire x1="96.52" y1="-99.06" x2="73.66" y2="-99.06" width="0.1524" layer="91"/>
+<label x="73.66" y="-99.06" size="1.778" layer="95" rot="R180" xref="yes"/>
+<pinref part="X1" gate="G$1" pin="-8"/>
+<wire x1="96.52" y1="-99.06" x2="99.06" y2="-99.06" width="0.1524" layer="91"/>
+<junction x="96.52" y="-99.06"/>
+</segment>
+<segment>
+<pinref part="IC4" gate="G$1" pin="A"/>
+<wire x1="111.76" y1="-20.32" x2="119.38" y2="-20.32" width="0.1524" layer="91"/>
+<label x="119.38" y="-20.32" size="1.778" layer="95" xref="yes"/>
+</segment>
+</net>
+<net name="DMX-" class="0">
+<segment>
+<pinref part="X1" gate="G$1" pin="B-9"/>
+<wire x1="96.52" y1="-101.6" x2="83.82" y2="-101.6" width="0.1524" layer="91"/>
+<label x="83.82" y="-101.6" size="1.778" layer="95" rot="R180" xref="yes"/>
+<pinref part="X1" gate="G$1" pin="-9"/>
+<wire x1="96.52" y1="-101.6" x2="99.06" y2="-101.6" width="0.1524" layer="91"/>
+<junction x="96.52" y="-101.6"/>
+</segment>
 <segment>
 <pinref part="IC4" gate="G$1" pin="B"/>
-<pinref part="U$2" gate="G$1" pin="1"/>
-<wire x1="111.76" y1="-22.86" x2="119.38" y2="-22.86" width="0.1524" layer="91"/>
-<wire x1="119.38" y1="-22.86" x2="129.54" y2="-12.7" width="0.1524" layer="91"/>
-</segment>
-</net>
-<net name="N$24" class="0">
-<segment>
-<pinref part="IC4" gate="G$1" pin="A"/>
-<pinref part="U$2" gate="G$1" pin="2"/>
-<wire x1="111.76" y1="-20.32" x2="129.54" y2="-20.32" width="0.1524" layer="91"/>
-</segment>
-</net>
+<wire x1="111.76" y1="-22.86" x2="129.54" y2="-22.86" width="0.1524" layer="91"/>
+<label x="129.54" y="-22.86" size="1.778" layer="95" xref="yes"/>
+</segment>
+</net>
+<net name="MOTOR+" class="0">
+<segment>
+<pinref part="X1" gate="G$1" pin="B-11"/>
+<label x="73.66" y="-106.68" size="1.778" layer="95" rot="R180" xref="yes"/>
+<wire x1="73.66" y1="-106.68" x2="96.52" y2="-106.68" width="0.1524" layer="91"/>
+<pinref part="X1" gate="G$1" pin="-11"/>
+<wire x1="96.52" y1="-106.68" x2="99.06" y2="-106.68" width="0.1524" layer="91"/>
+<junction x="96.52" y="-106.68"/>
+</segment>
+</net>
+<net name="MOTOR-" class="0">
+<segment>
+<pinref part="X1" gate="G$1" pin="B-12"/>
+<label x="86.36" y="-109.22" size="1.778" layer="95" rot="R180" xref="yes"/>
+<wire x1="96.52" y1="-109.22" x2="86.36" y2="-109.22" width="0.1524" layer="91"/>
+<pinref part="X1" gate="G$1" pin="-12"/>
+<wire x1="99.06" y1="-109.22" x2="96.52" y2="-109.22" width="0.1524" layer="91"/>
+<junction x="96.52" y="-109.22"/>
+</segment>
+</net>
